File: PCB_Schematic.kicad_sch (KiCad schematic)
At the start: 47 parts, among them J1 IMU_1, J2 Power_Connector, J3 Conn_02x05_Odd_Even, J6 USB_A, J7 Ultrasonic, J8 IMU_2, Q7 BSS138, SW1 SW_Push, U2 LM1117MP-ADJ, U3 TPS54331-Q1, U5 FT232RL, U6 STM32F091RCTx

Commit message: Sam
Parts:
- added FB1: FerriteBead, Inductor_SMD:L_0201_0603Metric_Pad0.64x0.40mm_HandSolder, symbol Device:FerriteBead
- added TP1: 3.3V TP, symbol Connector:TestPoint
- added TP2: 5V TP, symbol Connector:TestPoint
- added TP3: Echo TP, symbol Connector:TestPoint
- added U1: MAX7375AXR805, Package_TO_SOT_SMD:SOT-323_SC-70, symbol Oscillator:MAX7375AXR805
Connections:
- net +3.3V: now also TP1.1, U1.1 (V+)
- net +5V: now also FB1.2; no longer C3.1, C4.1
- net GND: now also U1.3 (GND)
- net Echo3.3V: now reaches Q7.2 (S), R3.2
- net Echo3.3V: now also U6.59 (PB7), TP3.1
- net at D4.1 (K), D8.2 (A): now also TP2.1
- net BOOT0: no longer names the net of U6.60 (PF11)
- net Echo renamed Echo5V
- net Echo5V: no longer U6.59 (PB7)
- new net: C3.1, C4.1, FB1.1
- no-connect marks 63 -> 61
Other:
- note added: "Connectors"
- note added: "Power Circuitry (Buck/LDO/Decoupling Caps)"
- note added: "Reset Switch/External Oscillator/Programming Header"
- note added: "STM32"
- note added: "USB to UART Converter"
- moved on the sheet: C1, C14, C2, C3, C4, C5, C6, C7, C8, C9, Cboot1, Ccomp1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

Commit message: Sam
Parts:
- added C10: .1 uF, Capacitor_SMD:C_1206_3216Metric_Pad1.33x1.80mm_HandSolder, symbol Device:C
- added D5, D6: LED_Blue, LED_SMD:LED_0805_2012Metric_Pad1.15x1.40mm_HandSolder, symbol Device:LED
- added H1, H2, H3, H4: MountingHole, MountingHole:MountingHole_2.2mm_M2, symbol Mechanical:MountingHole
- added J4: Conn_01x02_Pin, Connector_AMASS:AMASS_XT30PW-M_1x02_P2.50mm_Horizontal, symbol Connector:Conn_01x02_Pin
- added R10, R7: 10k, Resistor_SMD:R_0805_2012Metric_Pad1.20x1.40mm_HandSolder, symbol Device:R_US
- C6: footprint Capacitor_SMD:C_1206_3216Metric_Pad1.33x1.80mm_HandSolder -> Capacitor_SMD:C_0805_2012Metric_Pad1.18x1.45mm_HandSolder
- D2, D3: value LED -> LED_Blue; footprint (none) -> LED_SMD:LED_0805_2012Metric_Pad1.15x1.40mm_HandSolder
- D7: value LED -> LED_Red; footprint (none) -> LED_SMD:LED_0805_2012Metric_Pad1.15x1.40mm_HandSolder
- R1, R2, R5, R8: footprint Resistor_SMD:R_1206_3216Metric_Pad1.30x1.75mm_HandSolder -> Resistor_SMD:R_0805_2012Metric_Pad1.20x1.40mm_HandSolder
Connections:
- net +3.3V: now also C10.1, R7.2
- net +5V: now also R10.2
- net GND: now also C10.2, D5.1 (K), D6.1 (K)
- net PC0: now also J4.1 (Pin_1)
- net PC1: now also J4.2 (Pin_2)
- net PC14: now also U1.2 (CLOCK)
- new net: D6.2 (A), R10.1
- new net: D5.2 (A), R7.1
- no-connect marks 61 -> 58
Other:
- note added: "Connector Header for extrs GPIOs"
- note added: "Power Indicators"

Commit message: more
Parts:
- removed C14: .1 uF, Capacitor_SMD:C_1206_3216Metric_Pad1.33x1.80mm_HandSolder, symbol Device:C
- removed R11: 100K, Resistor_SMD:R_1206_3216Metric_Pad1.30x1.75mm_HandSolder, symbol Device:R
- added C11: .1uF, Capacitor_SMD:C_0805_2012Metric_Pad1.18x1.45mm_HandSolder, symbol Device:C
- added R11: 100K, Resistor_SMD:R_0805_2012Metric_Pad1.20x1.40mm_HandSolder, symbol Device:R_US
- D1, D4: value D_Schottky -> BAT60JFILM; footprint (none) -> Diode_SMD:D_0805_2012Metric_Pad1.15x1.40mm_HandSolder
- D8: value LED -> LED_Blue; footprint (none) -> LED_SMD:LED_0805_2012Metric_Pad1.15x1.40mm_HandSolder
- J3: footprint (none) -> Connector_IDC:IDC-Header_2x05_P2.54mm_Vertical
- R3, R4: footprint Resistor_SMD:R_1206_3216Metric_Pad1.30x1.75mm_HandSolder -> Resistor_SMD:R_0805_2012Metric_Pad1.20x1.40mm_HandSolder
- R6: footprint Resistor_SMD:R_1206_3216Metric_Pad1.30x1.75mm_HandSolder -> Capacitor_SMD:C_0805_2012Metric_Pad1.18x1.45mm_HandSolder
- SW1: footprint (none) -> Button_Switch_SMD:SW_SPST_PTS645
Connections:
- net +3.3V: now also R11.1
- net GND: now also C11.2
- net NRST: now also C11.1, R11.2

Commit message: More changes
Parts:
- L1: footprint (none) -> Inductor_SMD:L_1206_3216Metric
Changed lines of the file:
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@@
 			)
 		)
-		(property "Footprint" ""
+		(property "Footprint" "Inductor_SMD:L_1206_3216Metric"
 			(at 130.81 135.89 0)
 			(effects

Commit message: cookies
Parts:
- added C12: 4.7 uF, Capacitor_SMD:C_1206_3216Metric_Pad1.33x1.80mm_HandSolder, symbol Device:C
- added C13: 10 uF, Capacitor_SMD:C_1206_3216Metric_Pad1.33x1.80mm_HandSolder, symbol Device:C
- J3: value Conn_02x05_Odd_Even -> Programming Header
- SW1: value SW_Push -> Reset Switch
- TP1, TP2, TP3: footprint (none) -> TestPoint:TestPoint_Loop_D3.50mm_Drill1.4mm_Beaded
Connections:
- net +3.3V: now also C12.1, C13.1
- net GND: now also C12.2, C13.2
- net PC12 renamed RXD
- net PD2 renamed TXD
Other:
- moved on the sheet: C10, C11, C3, C4, C5, FB1, J3, J4, R10, R11, R5, R6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

Commit message: no errors
Changed lines of the file:
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@@
 	)
 	(junction
+		(at 137.16 186.69)
+		(diameter 0)
+		(color 0 0 0 0)
+	)
+	(junction
 		(at 93.98 186.69)
 		(diameter 0)
@@
 	)
 	(symbol
+		(lib_id "power:PWR_FLAG")
+		(at 57.15 26.67 270)
+		(unit 1)
+		(exclude_from_sim no)
+		(in_bom yes)
+		(on_board yes)
+		(dnp no)
+		(property "Reference" "#FLG01"
+			(at 59.055 26.67 0)
+			(effects
+				(font
+					(size 1.27 1.27)
+				)
+				(hide yes)
+			)
+		)
+		(property "Value" "PWR_FLAG"
+			(at 59.69 27.94 90)
+			(effects
+				(font
+					(size 1.27 1.27)
+				)
+				(justify left)
+			)
+		)
+		(property "Footprint" ""
+			(at 57.15 26.67 0)
+			(effects
+				(font
+					(size 1.27 1.27)
+				)
+				(hide yes)
+			)
+		)
+		(property "Datasheet" "~"
+			(at 57.15 26.67 0)
+			(effects
+				(font
+					(size 1.27 1.27)
+				)
+				(hide yes)
+			)
+		)
+		(property "Description" "Special symbol for telling ERC where power comes from"
+			(at 57.15 26.67 0)
+			(effects
+				(font
+					(size 1.27 1.27)
+				)
+				(hide yes)
+			)
+		)
+		(pin "1"
+		)
+		(instances
+			(project ""
+				(path "/a0c17764-e0d1-4df5-b871-1489cf266494"
+					(reference "#FLG01")
+					(unit 1)
+				)
+			)
+		)
+	)
+	(symbol
 		(lib_id "power:+5V")
 		(at 55.88 101.6 0)
@@
 	)
 	(symbol
+		(lib_id "power:PWR_FLAG")
+		(at 137.16 186.69 180)
+		(unit 1)
+		(exclude_from_sim no)
+		(in_bom yes)
+		(on_board yes)
+		(dnp no)
+		(fields_autoplaced yes)
+		(property "Reference" "#FLG02"
+			(at 137.16 188.595 0)
+			(effects
+				(font
+					(size 1.27 1.27)
+				)
+				(hide yes)
+			)
+		)
+		(property "Value" "PWR_FLAG"
+			(at 137.16 191.77 0)
+			(effects
+				(font
+					(size 1.27 1.27)
+				)
+			)
+		)
+		(property "Footprint" ""
+			(at 137.16 186.69 0)
+			(effects
+				(font
+					(size 1.27 1.27)
+				)
+				(hide yes)
+			)
+		)
+		(property "Datasheet" "~"
+			(at 137.16 186.69 0)
+			(effects
+				(font
+					(size 1.27 1.27)
+				)
+				(hide yes)
+			)
+		)
+		(property "Description" "Special symbol for telling ERC where power comes from"
+			(at 137.16 186.69 0)
+			(effects
+				(font
+					(size 1.27 1.27)
+				)
+				(hide yes)
+			)
+		)
+		(pin "1"
+		)
+		(instances
+			(project "PCB_Schematic"
+				(path "/a0c17764-e0d1-4df5-b871-1489cf266494"
+					(reference "#FLG02")
+					(unit 1)
+				)
+			)
+		)
+	)
+	(symbol
 		(lib_id "power:GND")
 		(at 264.16 119.38 90)
@@
 		(on_board yes)
 		(dnp no)
-		(fields_autoplaced yes)
 		(property "Reference" "U5"
-			(at 59.1694 26.67 0)
+			(at 60.96 30.48 0)
 			(effects
 				(font
@@
 		)
 		(property "Value" "FT232RL"
-			(at 59.1694 29.21 0)
+			(at 64.008 30.226 0)
 			(effects
 				(font

Commit message: new caps
Parts:
- removed C1, Cin1: 10 uF, Capacitor_SMD:C_1206_3216Metric_Pad1.33x1.80mm_HandSolder, symbol Device:C_Polarized_US
- removed C2: 100 uF, Capacitor_SMD:C_1206_3216Metric_Pad1.33x1.80mm_HandSolder, symbol Device:C_Polarized_US
- removed C3, C5, Cboot1: 100 nF, Capacitor_SMD:C_1206_3216Metric_Pad1.33x1.80mm_HandSolder, symbol Device:C_Polarized_US
- removed C4: 4.7 uF, Capacitor_SMD:C_1206_3216Metric_Pad1.33x1.80mm_HandSolder, symbol Device:C_Polarized_US
- removed Ccomp1: 2.7 nF, Capacitor_SMD:C_1206_3216Metric_Pad1.33x1.80mm_HandSolder, symbol Device:C_Polarized_US
- removed Ccomp2: 10 pF, Capacitor_SMD:C_1206_3216Metric_Pad1.33x1.80mm_HandSolder, symbol Device:C_Polarized_US
- removed Cout1: 47 uF, symbol Device:C_Polarized_US
- removed Css1: 8.2 nF, Capacitor_SMD:C_1206_3216Metric_Pad1.33x1.80mm_HandSolder, symbol Device:C_Polarized_US
- added C1, Cin1: 10 uF, symbol Device:C
- added C2: 100 uF, symbol Device:C
- added C3, C5, Cboot1: 100 nF, symbol Device:C
- added C4: 4.7 uF, symbol Device:C
- added Ccomp1: 2.7 nF, symbol Device:C
- added Ccomp2: 10 pF, symbol Device:C
- added Cout1: 47 uF, symbol Device:C
- added Css1: 8.2 nF, symbol Device:C
Connections:
- net +3.3V: now also C2.1, Cout1.1
- net +5V: now also C1.1, Cin1.1
- net GND: now also C1.2, C2.2, C3.2, C4.2, C5.2, Ccomp1.2, Ccomp2.2, Cin1.2, Cout1.2, Css1.2
- net at U5.17 (3V3OUT), U5.4 (VCCIO): now also C5.1
- net at U3.8 (SS): now also Css1.1
- net at D1.1 (K), L1.1, U3.3 (PH): now also Cboot1.2
- net at U3.1 (BOOT): now also Cboot1.1
- net at Rcomp1.1, U3.6 (COMP): now also Ccomp2.1
- net at Rcomp1.2: now also Ccomp1.1
- net at FB1.1: now also C3.1, C4.1

Commit message: 1206 changed 0805
Parts:
- C10, C12, C13, C7, C8, C9: footprint Capacitor_SMD:C_1206_3216Metric_Pad1.33x1.80mm_HandSolder -> Capacitor_SMD:C_0805_2012Metric_Pad1.18x1.45mm_HandSolder
- C3, C4, C5, Cboot1, Ccomp1, Ccomp2, Cin1, Cout1, Css1: footprint (none) -> Capacitor_SMD:C_0805_2012Metric_Pad1.18x1.45mm_HandSolder
- L1: footprint Inductor_SMD:L_1206_3216Metric -> Inductor_SMD:L_0805_2012Metric_Pad1.15x1.40mm_HandSolder
- R9, Rcomp1, Rfbb1, Rfbt1: footprint Resistor_SMD:R_1206_3216Metric_Pad1.30x1.75mm_HandSolder -> Resistor_SMD:R_0805_2012Metric_Pad1.20x1.40mm_HandSolder
Changed lines of the file:
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@@
 			)
 		)
-		(property "Footprint" "Capacitor_SMD:C_1206_3216Metric_Pad1.33x1.80mm_HandSolder"
+		(property "Footprint" "Capacitor_SMD:C_0805_2012Metric_Pad1.18x1.45mm_HandSolder"
 			(at 94.9452 186.69 0)
 			(effects
@@
 			)
 		)
-		(property "Footprint" "Capacitor_SMD:C_1206_3216Metric_Pad1.33x1.80mm_HandSolder"
+		(property "Footprint" "Capacitor_SMD:C_0805_2012Metric_Pad1.18x1.45mm_HandSolder"
 			(at 106.3752 186.69 0)
 			(effects
@@
 			)
 		)
-		(property "Footprint" "Capacitor_SMD:C_1206_3216Metric_Pad1.33x1.80mm_HandSolder"
+		(property "Footprint" "Capacitor_SMD:C_0805_2012Metric_Pad1.18x1.45mm_HandSolder"
 			(at 138.1252 186.69 0)
 			(effects
@@
 			)
 		)
-		(property "Footprint" ""
+		(property "Footprint" "Capacitor_SMD:C_0805_2012Metric_Pad1.18x1.45mm_HandSolder"
 			(at 20.0152 43.18 0)
 			(effects
@@
 			)
 		)
-		(property "Footprint" ""
+		(property "Footprint" "Capacitor_SMD:C_0805_2012Metric_Pad1.18x1.45mm_HandSolder"
 			(at 30.1752 152.4 0)
 			(effects
@@
 			)
 		)
-		(property "Footprint" "Capacitor_SMD:C_1206_3216Metric_Pad1.33x1.80mm_HandSolder"
+		(property "Footprint" "Capacitor_SMD:C_0805_2012Metric_Pad1.18x1.45mm_HandSolder"
 			(at 116.5352 186.69 0)
 			(effects
@@
 			)
 		)
-		(property "Footprint" "Resistor_SMD:R_1206_3216Metric_Pad1.30x1.75mm_HandSolder"
+		(property "Footprint" "Resistor_SMD:R_0805_2012Metric_Pad1.20x1.40mm_HandSolder"
 			(at 170.18 137.668 90)
 			(effects
@@
 			)
 		)
-		(property "Footprint" ""
+		(property "Footprint" "Capacitor_SMD:C_0805_2012Metric_Pad1.18x1.45mm_HandSolder"
 			(at 159.7152 149.86 0)
 			(effects
@@
 			)
 		)
-		(property "Footprint" ""
+		(property "Footprint" "Capacitor_SMD:C_0805_2012Metric_Pad1.18x1.45mm_HandSolder"
 			(at 55.5752 152.4 0)
 			(effects
@@
 			)
 		)
-		(property "Footprint" "Inductor_SMD:L_1206_3216Metric"
+		(property "Footprint" "Inductor_SMD:L_0805_2012Metric_Pad1.15x1.40mm_HandSolder"
 			(at 130.81 135.89 0)
 			(effects
@@
 			)
 		)
-		(property "Footprint" ""
+		(property "Footprint" "Capacitor_SMD:C_0805_2012Metric_Pad1.18x1.45mm_HandSolder"
 			(at 74.6252 24.13 0)
 			(effects
@@
 			)
 		)
-		(property "Footprint" ""
+		(property "Footprint" "Capacitor_SMD:C_0805_2012Metric_Pad1.18x1.45mm_HandSolder"
 			(at 17.4752 152.4 0)
 			(effects
@@
 			)
 		)
-		(property "Footprint" ""
+		(property "Footprint" "Capacitor_SMD:C_0805_2012Metric_Pad1.18x1.45mm_HandSolder"
 			(at 108.9152 133.35 0)
 			(effects
@@
 			)
 		)
-		(property "Footprint" ""
+		(property "Footprint" "Capacitor_SMD:C_0805_2012Metric_Pad1.18x1.45mm_HandSolder"
 			(at 63.1952 24.13 0)
 			(effects
@@
 			)
 		)
-		(property "Footprint" "Resistor_SMD:R_1206_3216Metric_Pad1.30x1.75mm_HandSolder"
+		(property "Footprint" "Resistor_SMD:R_0805_2012Metric_Pad1.20x1.40mm_HandSolder"
 			(at 141.732 151.13 90)
 			(effects
@@
 			)
 		)
-		(property "Footprint" "Resistor_SMD:R_1206_3216Metric_Pad1.30x1.75mm_HandSolder"
+		(property "Footprint" "Resistor_SMD:R_0805_2012Metric_Pad1.20x1.40mm_HandSolder"
 			(at 40.132 139.7 90)
 			(effects
@@
 			)
 		)
-		(property "Footprint" "Resistor_SMD:R_1206_3216Metric_Pad1.30x1.75mm_HandSolder"
+		(property "Footprint" "Resistor_SMD:R_0805_2012Metric_Pad1.20x1.40mm_HandSolder"
 			(at 141.732 139.7 90)
 			(effects
@@
 			)
 		)
-		(property "Footprint" "Capacitor_SMD:C_1206_3216Metric_Pad1.33x1.80mm_HandSolder"
+		(property "Footprint" "Capacitor_SMD:C_0805_2012Metric_Pad1.18x1.45mm_HandSolder"
 			(at 126.6952 186.69 0)
 			(effects
@@
 			)
 		)
-		(property "Footprint" ""
+		(property "Footprint" "Capacitor_SMD:C_0805_2012Metric_Pad1.18x1.45mm_HandSolder"
 			(at 42.8752 152.4 0)
 			(effects
@@
 			)
 		)
-		(property "Footprint" "Capacitor_SMD:C_1206_3216Metric_Pad1.33x1.80mm_HandSolder"
+		(property "Footprint" "Capacitor_SMD:C_0805_2012Metric_Pad1.18x1.45mm_HandSolder"
 			(at 198.12 73.3552 0)
 			(effects
