File: USB_UART_subsheet.kicad_sch (KiCad schematic)
At the start: 10 parts, among them U2 FT232RL

Commit message: done fr
Connections:
- net +5V: no longer U2.19 (~{RESET})
- net Vcc: now also U2.19 (~{RESET})
Changed lines of the file:
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@@
 	(paper "A4")
 	(junction
-		(at 146.05 78.74)
+		(at 146.05 77.47)
+		(diameter 0)
+		(color 0 0 0 0)
+	)
+	(junction
+		(at 146.05 74.93)
 		(diameter 0)
 		(color 0 0 0 0)
@@
 	(wire
 		(pts
+			(xy 93.98 73.66) (xy 134.62 73.66)
+		)
+		(stroke
+			(width 0)
+			(type default)
+		)
+	)
+	(wire
+		(pts
 			(xy 146.05 130.81) (xy 148.59 130.81)
 		)
@@
 	(wire
 		(pts
-			(xy 146.05 72.39) (xy 146.05 78.74)
+			(xy 146.05 72.39) (xy 146.05 74.93)
 		)
 		(stroke
@@
 	(wire
 		(pts
+			(xy 93.98 105.41) (xy 93.98 73.66)
+		)
+		(stroke
+			(width 0)
+			(type default)
+		)
+	)
+	(wire
+		(pts
 			(xy 146.05 72.39) (xy 226.06 72.39)
 		)
@@
 	(wire
 		(pts
+			(xy 146.05 77.47) (xy 146.05 80.01)
+		)
+		(stroke
+			(width 0)
+			(type default)
+		)
+	)
+	(wire
+		(pts
 			(xy 121.92 87.63) (xy 121.92 80.01)
 		)
@@
 	(wire
 		(pts
+			(xy 93.98 105.41) (xy 123.19 105.41)
+		)
+		(stroke
+			(width 0)
+			(type default)
+		)
+	)
+	(wire
+		(pts
 			(xy 143.51 130.81) (xy 146.05 130.81)
 		)
@@
 	(wire
 		(pts
-			(xy 152.4 74.93) (xy 152.4 78.74)
-		)
-		(stroke
-			(width 0)
-			(type default)
-		)
-	)
-	(wire
-		(pts
 			(xy 180.34 111.76) (xy 180.34 115.57)
 		)
@@
 	(wire
 		(pts
-			(xy 118.11 105.41) (xy 123.19 105.41)
-		)
-		(stroke
-			(width 0)
-			(type default)
-		)
-	)
-	(wire
-		(pts
 			(xy 166.37 82.55) (xy 172.72 82.55)
 		)
@@
 	(wire
 		(pts
+			(xy 134.62 73.66) (xy 134.62 77.47)
+		)
+		(stroke
+			(width 0)
+			(type default)
+		)
+	)
+	(wire
+		(pts
 			(xy 107.95 87.63) (xy 121.92 87.63)
 		)
@@
 	(wire
 		(pts
-			(xy 152.4 78.74) (xy 146.05 78.74)
-		)
-		(stroke
-			(width 0)
-			(type default)
-		)
-	)
-	(wire
-		(pts
-			(xy 152.4 74.93) (xy 166.37 74.93)
+			(xy 146.05 74.93) (xy 166.37 74.93)
+		)
+		(stroke
+			(width 0)
+			(type default)
+		)
+	)
+	(wire
+		(pts
+			(xy 134.62 77.47) (xy 146.05 77.47)
 		)
 		(stroke
@@
 	(wire
 		(pts
-			(xy 146.05 78.74) (xy 146.05 80.01)
+			(xy 146.05 74.93) (xy 146.05 77.47)
 		)
 		(stroke
@@
 					(unit 1)
 				)
-			)
-		)
-	)
-	(symbol
-		(lib_id "power:+5V")
-		(at 118.11 105.41 0)
-		(unit 1)
-		(exclude_from_sim no)
-		(in_bom yes)
-		(on_board yes)
-		(dnp no)
-		(fields_autoplaced yes)
-		(property "Reference" "#PWR013"
-			(at 118.11 109.22 0)
-			(effects
-				(font
-					(size 1.27 1.27)
-				)
-				(hide yes)
-			)
-		)
-		(property "Value" "+5V"
-			(at 118.11 100.33 0)
-			(effects
-				(font
-					(size 1.27 1.27)
-				)
-			)
-		)
-		(property "Footprint" ""
-			(at 118.11 105.41 0)
-			(effects
-				(font
-					(size 1.27 1.27)
-				)
-				(hide yes)
-			)
-		)
-		(property "Datasheet" ""
-			(at 118.11 105.41 0)
-			(effects
-				(font
-					(size 1.27 1.27)
-				)
-				(hide yes)
-			)
-		)
-		(property "Description" "Power symbol creates a global label with name \"+5V\""
-			(at 118.11 105.41 0)
-			(effects
-				(font
-					(size 1.27 1.27)
-				)
-				(hide yes)
-			)
-		)
-		(pin "1"
-		)
-		(instances
-			(project "PCB_Schematic"
-				(path "/a0c17764-e0d1-4df5-b871-1489cf266494/8edd1d5f-65c6-4da1-89c4-ae03b62a6366"
-					(reference "#PWR013")
-					(unit 1)
-				)
