File: Power_subsheet.kicad_sch (KiCad schematic)
At the start: 30 parts, among them U3 LM1117MP-ADJ, U4 TPS54331QDRQ1

Commit message: more changes
Parts:
- Cboot1, Rcomp1, Rfbb1, Rfbt1: footprint Capacitor_SMD:C_0402_1005Metric_Pad0.74x0.62mm_HandSolder -> Resistor_SMD:R_0805_2012Metric_Pad1.20x1.40mm_HandSolder
- Cin1, Cout1: footprint Capacitor_SMD:C_1210_3225Metric_Pad1.33x2.70mm_HandSolder -> Capacitor_SMD:C_0805_2012Metric_Pad1.18x1.45mm_HandSolder
- Css1: footprint Capacitor_SMD:C_0201_0603Metric -> Capacitor_SMD:C_0805_2012Metric_Pad1.18x1.45mm_HandSolder
Changed lines of the file:
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@@
 			)
 		)
-		(property "Footprint" "Capacitor_SMD:C_0402_1005Metric_Pad0.74x0.62mm_HandSolder"
+		(property "Footprint" "Resistor_SMD:R_0805_2012Metric_Pad1.20x1.40mm_HandSolder"
 			(at 70.612 80.01 90)
 			(effects
@@
 			)
 		)
-		(property "Footprint" "Capacitor_SMD:C_0201_0603Metric"
+		(property "Footprint" "Capacitor_SMD:C_0805_2012Metric_Pad1.18x1.45mm_HandSolder"
 			(at 86.0552 92.71 0)
 			(effects
@@
 			)
 		)
-		(property "Footprint" "Capacitor_SMD:C_0402_1005Metric_Pad0.74x0.62mm_HandSolder"
+		(property "Footprint" "Resistor_SMD:R_0805_2012Metric_Pad1.20x1.40mm_HandSolder"
 			(at 215.392 82.55 90)
 			(effects
@@
 			)
 		)
-		(property "Footprint" "Capacitor_SMD:C_1210_3225Metric_Pad1.33x2.70mm_HandSolder"
+		(property "Footprint" "Capacitor_SMD:C_0805_2012Metric_Pad1.18x1.45mm_HandSolder"
 			(at 47.9552 92.71 0)
 			(effects
@@
 			)
 		)
-		(property "Footprint" "Capacitor_SMD:C_0402_1005Metric_Pad0.74x0.62mm_HandSolder"
+		(property "Footprint" "Resistor_SMD:R_0805_2012Metric_Pad1.20x1.40mm_HandSolder"
 			(at 215.392 71.12 90)
 			(effects
@@
 			)
 		)
-		(property "Footprint" "Capacitor_SMD:C_1210_3225Metric_Pad1.33x2.70mm_HandSolder"
+		(property "Footprint" "Capacitor_SMD:C_0805_2012Metric_Pad1.18x1.45mm_HandSolder"
 			(at 237.1852 81.28 0)
 			(effects
@@
 			)
 		)
-		(property "Footprint" "Capacitor_SMD:C_0402_1005Metric_Pad0.74x0.62mm_HandSolder"
+		(property "Footprint" "Resistor_SMD:R_0805_2012Metric_Pad1.20x1.40mm_HandSolder"
 			(at 107.6452 64.77 0)
 			(effects

Commit message: updated fp
Parts:
- removed TP3: 3.3V TP, TestPoint:TestPoint_Loop_D3.50mm_Drill1.4mm_Beaded, symbol Connector:TestPoint
- D11: footprint Diode_SMD:D_0805_2012Metric_Pad1.15x1.40mm_HandSolder -> Diode_SMD:D_SOD-323_HandSoldering
- D12: footprint Diode_SMD:D_SOD-123F -> Diode_SMD:D_SOD-123
Changed lines of the file:
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@@
 	)
 	(junction
-		(at 71.12 130.81)
-		(diameter 0)
-		(color 0 0 0 0)
-	)
-	(junction
 		(at 86.36 180.34)
 		(diameter 0)
@@
 	(wire
 		(pts
-			(xy 69.85 130.81) (xy 71.12 130.81)
+			(xy 69.85 130.81) (xy 76.2 130.81)
 		)
 		(stroke
@@
 	(wire
 		(pts
-			(xy 71.12 130.81) (xy 76.2 130.81)
-		)
-		(stroke
-			(width 0)
-			(type default)
-		)
-	)
-	(wire
-		(pts
 			(xy 59.69 92.71) (xy 72.39 92.71)
 		)
@@
 			)
 		)
-		(property "Footprint" "Diode_SMD:D_0805_2012Metric_Pad1.15x1.40mm_HandSolder"
+		(property "Footprint" "Diode_SMD:D_SOD-323_HandSoldering"
 			(at 66.04 130.81 0)
 			(effects
@@
 	)
 	(symbol
-		(lib_id "Connector:TestPoint")
-		(at 71.12 130.81 0)
-		(unit 1)
-		(exclude_from_sim no)
-		(in_bom yes)
-		(on_board yes)
-		(dnp no)
-		(fields_autoplaced yes)
-		(property "Reference" "TP3"
-			(at 73.66 126.2379 0)
-			(effects
-				(font
-					(size 1.27 1.27)
-				)
-				(justify left)
-			)
-		)
-		(property "Value" "3.3V TP"
-			(at 73.66 128.7779 0)
-			(effects
-				(font
-					(size 1.27 1.27)
-				)
-				(justify left)
-			)
-		)
-		(property "Footprint" "TestPoint:TestPoint_Loop_D3.50mm_Drill1.4mm_Beaded"
-			(at 76.2 130.81 0)
-			(effects
-				(font
-					(size 1.27 1.27)
-				)
-				(hide yes)
-			)
-		)
-		(property "Datasheet" "~"
-			(at 76.2 130.81 0)
-			(effects
-				(font
-					(size 1.27 1.27)
-				)
-				(hide yes)
-			)
-		)
-		(property "Description" "test point"
-			(at 71.12 130.81 0)
-			(effects
-				(font
-					(size 1.27 1.27)
-				)
-				(hide yes)
-			)
-		)
-		(pin "1"
-		)
-		(instances
-			(project "PCB_Schematic"
-				(path "/a0c17764-e0d1-4df5-b871-1489cf266494/e6fb26c7-dfd6-4c6c-883e-94dceb19958a"
-					(reference "TP3")
-					(unit 1)
-				)
-			)
-		)
-	)
-	(symbol
 		(lib_id "power:PWR_FLAG")
 		(at 54.61 69.85 0)
@@
 			)
 		)
-		(property "Footprint" "Diode_SMD:D_SOD-123F"
+		(property "Footprint" "Diode_SMD:D_SOD-123"
 			(at 198.12 71.12 0)
 			(effects

Commit message: footprint
Parts:
- renumbered D12 to D10, D13 to D11, D11 to D9, R12 to R10, R13 to R11, R14 to R12
Changed lines of the file:
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@@
 		(dnp no)
 		(fields_autoplaced yes)
-		(property "Reference" "R12"
+		(property "Reference" "R10"
 			(at 78.74 137.1599 0)
 			(effects
@@
 			(project "PCB_Schematic"
 				(path "/a0c17764-e0d1-4df5-b871-1489cf266494/e6fb26c7-dfd6-4c6c-883e-94dceb19958a"
-					(reference "R12")
+					(reference "R10")
 					(unit 1)
 				)
@@
 		(dnp no)
 		(fields_autoplaced yes)
-		(property "Reference" "R14"
+		(property "Reference" "R12"
 			(at 247.65 60.96 90)
 			(effects
@@
 			(project "PCB_Schematic"
 				(path "/a0c17764-e0d1-4df5-b871-1489cf266494/e6fb26c7-dfd6-4c6c-883e-94dceb19958a"
-					(reference "R14")
+					(reference "R12")
 					(unit 1)
 				)
@@
 		(dnp no)
 		(fields_autoplaced yes)
-		(property "Reference" "D13"
+		(property "Reference" "D11"
 			(at 241.6175 59.69 0)
 			(effects
@@
 			(project "PCB_Schematic"
 				(path "/a0c17764-e0d1-4df5-b871-1489cf266494/e6fb26c7-dfd6-4c6c-883e-94dceb19958a"
-					(reference "D13")
+					(reference "D11")
 					(unit 1)
 				)
@@
 		(on_board yes)
 		(dnp no)
-		(property "Reference" "D11"
+		(property "Reference" "D9"
 			(at 64.77 135.636 90)
 			(effects
@@
 			(project "PCB_Schematic"
 				(path "/a0c17764-e0d1-4df5-b871-1489cf266494/e6fb26c7-dfd6-4c6c-883e-94dceb19958a"
-					(reference "D11")
+					(reference "D9")
 					(unit 1)
 				)
@@
 		(on_board yes)
 		(dnp no)
-		(property "Reference" "D12"
+		(property "Reference" "D10"
 			(at 202.946 72.39 90)
 			(effects
@@
 			(project "PCB_Schematic"
 				(path "/a0c17764-e0d1-4df5-b871-1489cf266494/e6fb26c7-dfd6-4c6c-883e-94dceb19958a"
-					(reference "D12")
+					(reference "D10")
 					(unit 1)
 				)
@@
 		(dnp no)
 		(fields_autoplaced yes)
-		(property "Reference" "R13"
+		(property "Reference" "R11"
 			(at 78.74 149.8599 0)
 			(effects
@@
 			(project "PCB_Schematic"
 				(path "/a0c17764-e0d1-4df5-b871-1489cf266494/e6fb26c7-dfd6-4c6c-883e-94dceb19958a"
-					(reference "R13")
-					(unit 1)
-				)
+					(reference "R11")
+					(unit 1)
+				)

Commit message: buck
Connections:
- net PH: now reaches Cboot1.1, D10.1 (K), L1.1, U4.8 (PH)
Changed lines of the file:
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@@
+		)
+	)
+	(label "PH"
+		(at 180.34 67.31 0)
+		(fields_autoplaced yes)
+		(effects
+			(font
+				(size 1.27 1.27)
+			)
+			(justify left bottom)
+		)
+	)
+	(label "Vin"
+		(at 114.3 69.85 0)
+		(fields_autoplaced yes)
+		(effects
+			(font
+				(size 1.27 1.27)
+			)
+			(justify left bottom)
 		)
 	)

Commit message: changes
Parts:
- removed U3: LM1117MP-ADJ, Package_TO_SOT_SMD:SOT-223, symbol Regulator_Linear:LM1117MP-ADJ
- added U3: LM1117MP-ADJ, Library:REALWORKLDOFT, symbol New_Library:LM1117MP-ADJ
Connections:
- net +3.3V: now also U3.4 (VOUT)
- net +5V: now also U3.3 (IN)
- net at R10.2, R11.1: now also U3.1 (ADJ/GND)
- net at D9.2 (A): now also U3.2 (OUT)
Other:
- moved on the sheet: C4, D9

Commit message: final sending for review
Connections:
- net +3.3V: no longer U3.4 (VOUT)
- net at D9.2 (A), U3.2 (OUT): now also U3.4 (VOUT)
Changed lines of the file:
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@@
+	)
+	(junction
+		(at 66.04 130.81)
+		(diameter 0)
+		(color 0 0 0 0)
 	)
 	(junction
@@
 	(junction
 		(at 86.36 180.34)
-		(diameter 0)
-		(color 0 0 0 0)
-	)
-	(junction
-		(at 120.65 133.35)
 		(diameter 0)
 		(color 0 0 0 0)
@@
 	(wire
 		(pts
-			(xy 63.5 130.81) (xy 67.31 130.81)
+			(xy 63.5 130.81) (xy 66.04 130.81)
 		)
 		(stroke
@@
 	(wire
 		(pts
+			(xy 63.5 133.35) (xy 66.04 133.35)
+		)
+		(stroke
+			(width 0)
+			(type default)
+		)
+	)
+	(wire
+		(pts
 			(xy 184.15 67.31) (xy 189.23 67.31)
 		)
@@
 	(wire
 		(pts
-			(xy 63.5 133.35) (xy 120.65 133.35)
-		)
-		(stroke
-			(width 0)
-			(type default)
-		)
-	)
-	(wire
-		(pts
 			(xy 72.39 76.2) (xy 59.69 76.2)
 		)
@@
 	(wire
 		(pts
-			(xy 120.65 130.81) (xy 120.65 133.35)
+			(xy 120.65 130.81) (xy 120.65 135.89)
 		)
 		(stroke
@@
 	(wire
 		(pts
+			(xy 66.04 130.81) (xy 67.31 130.81)
+		)
+		(stroke
+			(width 0)
+			(type default)
+		)
+	)
+	(wire
+		(pts
 			(xy 208.28 81.28) (xy 208.28 77.47)
 		)
@@
 	(wire
 		(pts
-			(xy 120.65 133.35) (xy 120.65 135.89)
-		)
-		(stroke
-			(width 0)
-			(type default)
-		)
-	)
-	(wire
-		(pts
 			(xy 217.17 86.36) (xy 217.17 88.9)
 		)
 		(stroke
+			(width 0)
+			(type default)
+		)
+	)
+	(wire
+		(pts
+			(xy 66.04 130.81) (xy 66.04 133.35)
+		)
+		(stroke

Commit message: some changes
Parts:
- C10: value 10 nF -> .1uF
- C12, C9: value 4.7 uF -> .1uF
- C14: value 1 uF -> .1uF
- C5: value .1 uF -> 10nF
- C6, C8: value .1 uF -> 4.7uF
- C7: value .1 uF -> 1uF
Changed lines of the file:
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@@
 			)
 		)
-		(property "Value" ".1 uF"
+		(property "Value" "4.7uF"
 			(at 80.01 177.7999 0)
 			(effects
@@
 			)
 		)
-		(property "Value" "4.7 uF"
+		(property "Value" ".1uF"
 			(at 90.17 177.7999 0)
 			(effects
@@
 			)
 		)
-		(property "Value" "10 nF"
+		(property "Value" ".1uF"
 			(at 101.6 177.7999 0)
 			(effects
@@
 			)
 		)
-		(property "Value" "1 uF"
+		(property "Value" ".1uF"
 			(at 127 177.7999 0)
 			(effects
@@
 			)
 		)
-		(property "Value" ".1 uF"
+		(property "Value" "10nF"
 			(at 46.99 177.7999 0)
 			(effects
@@
 			)
 		)
-		(property "Value" ".1 uF"
+		(property "Value" "4.7uF"
 			(at 58.42 177.7999 0)
 			(effects
@@
 			)
 		)
-		(property "Value" ".1 uF"
+		(property "Value" "1uF"
 			(at 69.85 177.7999 0)
 			(effects
@@
 			)
 		)
-		(property "Value" "4.7 uF"
+		(property "Value" ".1uF"
 			(at 114.3 177.7999 0)
 			(effects
